File: 2.4GHzAmpAuto.kicad_pcb (KiCad board)
At the start: 2 copper layers, 55 x 72 mm, 40 parts, among them IC1 TLI4970, IC2 TLI4970, J1 MODULE CONNECTIONS, J10 program port, J2 OLED, J3 current A, J4 current B, J8 Fan1, J9 Fan2, SW1 SW_Push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

Commit message: Add files via upload
Parts:
- added REF**: MountingHole_2.5mm_Pad, MountingHole:MountingHole_2.5mm_Pad, F.Cu at (155.0, 89.8)
- added REF**: MountingHole_2.5mm_Pad, MountingHole:MountingHole_2.5mm_Pad, F.Cu at (155.0, 153.0)
- added REF**: MountingHole_2.5mm_Pad, MountingHole:MountingHole_2.5mm_Pad, F.Cu at (107.0, 153.0)
- added REF**: MountingHole_2.5mm_Pad, MountingHole:MountingHole_2.5mm_Pad, F.Cu at (107.0, 89.8)
- moved C1 5.16 mm to (110.8, 94.6)
- moved R9 5.00 mm to (111.0, 93.0)
- moved D2 2.17 mm to (121.0, 93.6), turned to 0 degrees
- moved J3 1.22 mm to (140.2, 88.6)
- moved J4 1.02 mm to (124.6, 88.6)
- moved R8 0.80 mm to (118.2, 91.0), turned to 180 degrees
- moved GND_IN1 0.30 mm to (113.3, 88.6)
Routing:
- net Net-(C1-Pad1): track 51.8 -> 58.7 mm
- net Net-(D1-Pad2): track 105.2 -> 100.5 mm
- net Net-(D2-Pad2): track 28.9 -> 31.6 mm
- net /GND: track 335.2 -> 332.9 mm
- net /Vdd: track 38.0 -> 39.8 mm
- net Net-(IC2-Pad7): track 14.3 -> 15.8 mm
- added copper zone on B.Cu, net /GND
Other:
- board text added: "Fan/pre-amp connectors"
- board text removed: "Fan connectors"

Commit message: Add files via upload
Parts:
- removed REF** (x4): MountingHole_2.5mm_Pad, MountingHole:MountingHole_2.5mm_Pad
- added C5: 0u1, Capacitor_SMD:C_0805_2012Metric, F.Cu at (145.7, 140.0)
- added H1: MountingHole_Pad, MountingHole:MountingHole_2.7mm_M2.5_Pad, F.Cu at (106.6, 90.2)
- added H2: MountingHole_Pad, MountingHole:MountingHole_2.7mm_M2.5_Pad, F.Cu at (155.0, 90.2)
- added H3: MountingHole_Pad, MountingHole:MountingHole_2.7mm_M2.5_Pad, F.Cu at (106.6, 153.2)
- added H4: MountingHole_Pad, MountingHole:MountingHole_2.7mm_M2.5_Pad, F.Cu at (155.0, 153.2)
- added R17: K33, Resistor_SMD:R_0805_2012Metric_Pad1.15x1.40mm_HandSolder, F.Cu at (146.6, 147.4)
- added R18: 10K, Resistor_SMD:R_0805_2012Metric_Pad1.15x1.40mm_HandSolder, F.Cu at (142.1, 141.9)
- IC1, IC2: value TLI4970 -> TLI4970D025T5XUMA1
- J1: value MODULE CONNECTIONS -> conections to module
- moved R4 2.10 mm to (132.2, 149.0)
- moved D1 0.78 mm to (152.6, 98.8)
Connections:
- J1 pad 4: Net-(J1-Pad4) -> /GND
- J1 pad 5: Net-(J1-Pad5) -> /PTT
Routing:
- net Net-(C5-Pad1): track 0.00 -> 35.7 mm, vias 0 -> 2
- net /PTT: track 0.00 -> 22.1 mm, vias 0 -> 2
- net /GND: track 332.9 -> 354.9 mm
- net /T3: track 49.4 -> 44.7 mm
- net /+3v3: track 146.1 -> 149.9 mm
- net /VG2: track 11.5 -> 12.4 mm
Other:
- board text added: "Issue 1 -PTT"
- board text added: "PTT"
- board text removed: "Issue 1"
